File: GaugESP32.sch (KiCad schematic (older format))
At the start: 56 parts, among them J1 Conn_01x20, J2 Conn_01x20, J3 Conn_02x02_Counter_Clockwise, J3 JST-PH, J3 USB_OTG, Q1 BC847, Q1 MBT3946DW1T1, U1 ESP-32S, U2 FT231XS, U3 BQ24075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

Commit message: Minor fixes
Parts:
- J5: renamed from J3; value USB_OTG -> Micro USB-B
- renumbered J3 to J4, Q1 to Q2, R19 to R22, R18 to R9
Connections:
- net labels removed: IO37, IO38, SHIELD, VN, VP
- wire segments 308 -> 258
- no-connect marks 13 -> 16
Other:
- note added: "IO37 and IO38 are\nnot available on module"

Commit message: V2 with ESP32-PICO-D4, and initial board
Parts:
- removed U1: ESP-32S, Z_ESP32:ESP-32S, symbol ESP-32S
- added AE1: Antenna_Shield, RF_Antennas:Texas_SWRA117D_2.4GHz_Left, symbol Antenna_Shield
- added C13, C15: 0.1uF, Capacitors_SMD:C_0603, symbol C
- added C14: 10uF, Capacitors_SMD:C_0603, symbol C
- added C16: 4.7pF, Capacitors_SMD:C_0603, symbol C
- added C17: 2.7pF, Capacitors_SMD:C_0603, symbol C
- added L2: 1.6nH, Inductors_SMD:L_0603, symbol L
- added U1: ESP32PICO_D4, ESP32PICO:ESP32_PICO_D4, symbol ESP32PICO_D4
- D2: value GREEN -> YELLOW
- L1: footprint Inductors_NEOSID:Neosid_Inductor_SM0603CG -> Inductors_SMD:L_0603
- Q1: footprint TO_SOT_Packages_SMD:SOT-363 -> TO_SOT_Packages_SMD:SOT-363_SC-70-6
- U2: footprint SSOP-20 -> Housings_DFN_QFN:QFN-20-1EP_4x4mm_Pitch0.5mm
- U3: footprint (none) -> Housings_DFN_QFN:QFN-16-1EP_3x3mm_Pitch0.5mm
- Y1: footprint (none) -> Crystals:Crystal_SMD_0603-2pin_6.0x3.5mm
Connections:
- net labels added: +3.3VA, IO37, IO38, LNA
- wire segments 258 -> 283
- no-connect marks 16 -> 18
Other:
- note removed: "IO37 and IO38 are\nnot available on module"

Commit message: Main ESP32 components placement
Parts:
- Y1: footprint Crystals:Crystal_SMD_0603-2pin_6.0x3.5mm -> Crystals:Crystal_SMD_3215-2pin_3.2x1.5mm
Changed lines of the file:
@@
 F 0 "Y1" H 5500 3000 50  0000 C CNN
 F 1 "32.768kHz" H 5500 2800 50  0000 C CNN
-F 2 "Crystals:Crystal_SMD_0603-2pin_6.0x3.5mm" H 5500 2900 50  0001 C CNN
+F 2 "Crystals:Crystal_SMD_3215-2pin_3.2x1.5mm" H 5500 2900 50  0001 C CNN
 F 3 "" H 5500 2900 50  0001 C CNN
 	1    5500 2900

Commit message: Layout work
Parts:
- U2: footprint Housings_DFN_QFN:QFN-20-1EP_4x4mm_Pitch0.5mm -> Housings_SSOP:SSOP-20_5.3x7.2mm_Pitch0.65mm
Connections:
- wire segments 283 -> 286
Changed lines of the file:
@@
 F 0 "U2" H 3500 5950 50  0000 L CNN
 F 1 "FT231XS" H 4350 5950 50  0000 L CNN
-F 2 "Housings_DFN_QFN:QFN-20-1EP_4x4mm_Pitch0.5mm" H 4050 5150 50  0001 C CNN
+F 2 "Housings_SSOP:SSOP-20_5.3x7.2mm_Pitch0.65mm" H 4050 5150 50  0001 C CNN
 F 3 "" H 4050 5150 50  0001 C CNN
 	1    4050 5150
@@
 	6150 5750 6050 5750
 Wire Wire Line
-	6050 5750 6050 6100
+	6050 5650 6050 6100
 Wire Wire Line
 	6150 5850 6050 5850
@@
 Wire Notes Line
 	6150 4400 6150 4300
+Wire Wire Line
+	6150 5650 6050 5650
+Connection ~ 6050 5750
+Wire Wire Line
+	3550 7250 3550 7400
+Wire Wire Line
+	3550 7400 3450 7400
+Connection ~ 3450 7400
 $EndSCHEMATC
